File: VexQwiic.kicad_pcb (KiCad board)
At the start: 2 copper layers, 32 x 70 mm, 55 parts, among them CON1 MIKROBUS_HOST_CONN, J1 Qwiic_RA, J2 USB_C_Receptacle_USB2.0, J3 JST-SM-M-WS2812, SW1 BOOTSEL, SW2 RESET, U1 W25Q128JVS, U2 RP2040, U3 TPS563200, U4 NCP1117-3.3_SOT223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

Commit message: Last version w/ rp2040
Parts:
- moved CON1 8.91 mm to (137.9, 104.8)
- moved C10 7.60 mm to (174.4, 98.9)
- moved C13 7.60 mm to (174.4, 106.4)
- moved C15 7.60 mm to (174.4, 111.4)
- moved C16 7.60 mm to (174.4, 113.9)
- moved C17 7.60 mm to (178.4, 98.9)
- moved C18 7.60 mm to (146.7, 116.7)
- moved C20 7.60 mm to (154.0, 111.4)
- moved C21 7.60 mm to (157.5, 108.2)
- moved C22 7.60 mm to (152.5, 114.9)
- moved C23 7.60 mm to (152.5, 119.9)
- moved C9 7.60 mm to (170.4, 113.9)
- moved J3 7.60 mm to (157.3, 124.4)
- moved R10 7.60 mm to (153.3, 95.9)
- moved R9 7.60 mm to (151.7, 95.9)
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
Commit message: Version 1 complete & ordered.
Parts:
- removed 3V3: TP_3.3V, TestPoint:TestPoint_Pad_D1.5mm
- removed C10, C11, C12, C13, C14, C16, C17, C18, C19, C21, C9: 100nF, Capacitor_SMD:C_0603_1608Metric
- removed C15, C20: 1uF, Capacitor_SMD:C_0603_1608Metric
- removed C22, C23: 15pF, Capacitor_SMD:C_0603_1608Metric
- removed C7, C8: 10uF, Capacitor_SMD:C_0603_1608Metric
- removed D4, D5: D_Schottky, Diode_SMD:D_SOD-323_HandSoldering
- removed GND1: TP_GND, TestPoint:TestPoint_Pad_D1.5mm
- removed J2: USB_C_Receptacle_USB2.0, Connector_USB:USB_C_Receptacle_GCT_USB4085
- removed J3: JST-SM-M-WS2812, Connector_PinHeader_2.54mm:PinHeader_1x03_P2.54mm_Vertical
- removed R10, R9: 27.4, Resistor_SMD:R_0603_1608Metric
- removed R4: 1M, Resistor_SMD:R_0603_1608Metric
- removed R5, R6: 5.11K, Resistor_SMD:R_0603_1608Metric
- removed R7, R8: 1k, Resistor_SMD:R_0603_1608Metric
- removed SW1: BOOTSEL, Button_Switch_THT:SW_PUSH_6mm_H13mm
- removed SW2: RESET, Button_Switch_THT:SW_PUSH_6mm_H13mm
- removed U2: RP2040, Package_DFN_QFN:QFN-56-1EP_7x7mm_P0.4mm_EP3.2x3.2mm
- removed U4: NCP1117-3.3_SOT223, Package_TO_SOT_SMD:SOT-223-3_TabPin2
- removed VIN1: TP_12V, TestPoint:TestPoint_Pad_D1.5mm
- removed X1: ABM8-272-T3, pcb:ABM8-272-T3_ABR
- added G***: LOGO, LOGO, F.Cu at (159.6, 74.6)
- added G***: LOGO, LOGO, B.Cu at (149.3, 105.6)
- J1: value Qwiic_RA -> Screw_Terminal_3.5mm_2; footprint SparkFun-Connector:JST_SMD_1.0mm-4_RA -> SparkFun-Connector:Screw_Terminal_3.5mm-2
- U1: value W25Q128JVS -> Sparkfun-ProMicroRP2350; footprint Package_SO:SOIC-8_5.23x5.23mm_P1.27mm -> Sparkfun-ProMicro2350:Sparkfun-ProMicro2350
- moved J1 68.1 mm to (158.8, 54.7), turned to 180 degrees
- moved U1 20.2 mm to (158.3, 125.0), turned to 180 degrees
- moved R3 20.1 mm to (138.9, 79.4)
- moved U5 17.4 mm to (138.8, 84.1), turned to 90 degrees
- moved D1 11.9 mm to (158.9, 64.3), turned to -90 degrees
- moved D2 9.44 mm to (155.4, 64.3), turned to -90 degrees
- moved CON1 7.78 mm to (138.1, 97.1)
- moved CONN1 0.72 mm to (141.9, 56.0)
Connections:
- J1 pad 1: GND -> +5V
- J1 pad 2: +3.3V -> GND
- U1 pad 1: Net-(U1-~{CS}) -> /RS485_RX
- U1 pad 2: Net-(U1-DO(IO1)) -> GND
- U1 pad 3: Net-(U1-IO2) -> GND
- U1 pad 4: GND -> /RS485_MODE
- U1 pad 5: Net-(U1-DI(IO0)) -> unconnected-(U1-3-Pad5)
- U1 pad 6: /QSPI_SCLK -> /MKBUS_SDA
- U1 pad 7: Net-(U1-IO3) -> /MKBUS_SCL
- U1 pad 8: +3.3V -> /MKBUS_INT
Routing:
- net /RS485_TX: track 0.00 -> 46.7 mm
- net /RS485_RX: track 0.00 -> 41.7 mm
- net /RJ9_DB: track 0.00 -> 38.6 mm, vias 0 -> 1
- net /RJ9_DA: track 0.00 -> 34.8 mm, vias 0 -> 1
- net /RS485_MODE: track 0.00 -> 34.1 mm
- net /MKBUS_MOSI: track 0.00 -> 19.1 mm, vias 0 -> 1
- net GND: track 3.45 -> 19.7 mm, vias 4 -> 6
- net /MKBUS_TX: track 0.00 -> 12.3 mm
- net /MKBUS_RX: track 0.00 -> 11.5 mm, vias 0 -> 1
- net /MKBUS_AN: track 0.00 -> 10.9 mm
- net /MKBUS_MISO: track 0.00 -> 9.91 mm, vias 0 -> 1
- net /MKBUS_CS: track 0.00 -> 9.91 mm, vias 0 -> 1
- net /MKBUS_SDA: track 0.00 -> 4.87 mm
- net /MKBUS_SCL: track 0.00 -> 4.87 mm
- net /MKBUS_SCK: track 0.00 -> 4.83 mm
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- added copper zone on F.Cu, net +5V
Other:
- board size 32 x 70 mm -> 32 x 75 mm
- board text added: "5V 3A Max"
- board text added: "GND"
- board text added: "V5 IFace Expander V1.0 10/28/2024"
- board text added: "©Ryan McGee 2024"
