File: VexQwiic.kicad_sch (KiCad schematic)
At the start: 55 parts, among them CON1 MIKROBUS_HOST_CONN, J1 Qwiic_RA, J2 USB_C_Receptacle_USB2.0, J3 JST-SM-M-WS2812, SW1 BOOTSEL, SW2 RESET, U1 W25Q128JVS, U2 RP2040, U3 TPS563200, U4 NCP1117-3.3_SOT223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

Commit message: Version 1 complete & ordered.
Parts:
- removed 3V3: TP_3.3V, TestPoint:TestPoint_Pad_D1.5mm, symbol Connector:TestPoint
- removed C10, C11, C12, C13, C14, C16, C17, C18, C19, C21, C9: 100nF, Capacitor_SMD:C_0603_1608Metric, symbol Device:C
- removed C15, C20: 1uF, Capacitor_SMD:C_0603_1608Metric, symbol Device:C
- removed C22, C23: 15pF, Capacitor_SMD:C_0603_1608Metric, symbol Device:C
- removed C7, C8: 10uF, Capacitor_SMD:C_0603_1608Metric, symbol Device:C
- removed D4, D5: D_Schottky, Diode_SMD:D_SOD-323_HandSoldering, symbol Device:D_Schottky
- removed GND1: TP_GND, TestPoint:TestPoint_Pad_D1.5mm, symbol Connector:TestPoint
- removed J1: Qwiic_RA, SparkFun-Connector:JST_SMD_1.0mm-4_RA, symbol SparkFun-Connector:Qwiic_Right_Angle
- removed J2: USB_C_Receptacle_USB2.0, Connector_USB:USB_C_Receptacle_GCT_USB4085, symbol Connector:USB_C_Receptacle_USB2.0
- removed J3: JST-SM-M-WS2812, Connector_PinHeader_2.54mm:PinHeader_1x03_P2.54mm_Vertical, symbol Connector_Generic:Conn_01x03
- removed R10, R9: 27.4, Resistor_SMD:R_0603_1608Metric, symbol Device:R_US
- removed R4: 1M, Resistor_SMD:R_0603_1608Metric, symbol Device:R_US
- removed R5, R6: 5.11K, Resistor_SMD:R_0603_1608Metric, symbol Device:R_US
- removed R7, R8: 1k, Resistor_SMD:R_0603_1608Metric, symbol Device:R_US
- removed SW1: BOOTSEL, Button_Switch_THT:SW_PUSH_6mm_H13mm, symbol Switch:SW_Push
- removed SW2: RESET, Button_Switch_THT:SW_PUSH_6mm_H13mm, symbol Switch:SW_Push
- removed U1: W25Q128JVS, Package_SO:SOIC-8_5.23x5.23mm_P1.27mm, symbol Memory_Flash:W25Q128JVS
- removed U2: RP2040, Package_DFN_QFN:QFN-56-1EP_7x7mm_P0.4mm_EP3.2x3.2mm, symbol MCU_RaspberryPi:RP2040
- removed U4: NCP1117-3.3_SOT223, Package_TO_SOT_SMD:SOT-223-3_TabPin2, symbol Regulator_Linear:NCP1117-3.3_SOT223
- removed VIN1: TP_12V, TestPoint:TestPoint_Pad_D1.5mm, symbol Connector:TestPoint
- removed X1: ABM8-272-T3, pcb:ABM8-272-T3_ABR, symbol 2024-08-11_22-55-58:ABM8-272-T3
- added J1: Screw_Terminal_3.5mm_2, SparkFun-Connector:Screw_Terminal_3.5mm-2, symbol SparkFun-Connector:Screw_Terminal_3.5mm_2
- added U1: Sparkfun-ProMicroRP2350, Sparkfun-ProMicro2350:Sparkfun-ProMicro2350, symbol Sparkfun-ProMicro2350:Sparkfun-ProMicro2350
Connections:
- net +3.3V: now also U1.15 (3.3V)
- net +5V: now also J1.1 (Pin_1), U1.12 (RAW)
- net GND: now also J1.2 (Pin_2), U1.13 (GND), U1.2 (GND), U1.3 (GND)
- net MKBUS_AN: now also U1.19 (A0)
- net MKBUS_CS: now also U1.23 (21/SPI_CS)
- net MKBUS_INT: now also U1.8 (6)
- net MKBUS_MISO: now also U1.21 (20/SPI_POCI)
- net MKBUS_MOSI: now also U1.22 (23/SPI_PICO)
- net MKBUS_PWM: now also U1.9 (7)
- net MKBUS_RX: now also U1.11 (9/RX1)
- net MKBUS_SCK: now also U1.20 (22/SPI_SCK)
- net MKBUS_SCL: now also U1.7 (5)
- net MKBUS_SDA: now also U1.6 (4)
- net MKBUS_TX: now also U1.10 (8/TX1)
- net RS485_MODE: now also U1.4 (2)
- net RS485_RX: now also U1.1 (1/RX)
- net RS485_TX: now also U1.0 (0/TX)
- no-connect marks 2 -> 5
Other:
- note removed: "I2C0"
- note removed: "I2C1"
- note removed: "Note: Keep decoupling caps close to their pin!"
- note removed: "Notes: - Keep SPI flash close to avoid crosstalk - Usually there's a pullup here on BOOTSEL, this chip doesn't need it I guess. - Keep USB resistors close to RP2040"
- note removed: "PWM0A"
- note removed: "SPI1"
- note removed: "UART0"
- note removed: "UART1"
- moved on the sheet: C1, C2, C3, C4, C5, CON1, D3, L1, R1, R2, U3
